File: beaglebone-cape/beaglebone-cape.sch (EAGLE design)
At the start: 7 parts

Commit message: [BB] Updated cape schematic w/ real resistors
Parts:
- R1, R2, R3, R4: value 5K -> 4.7K
Other:
- note added: "Provided on Cape"
Changed lines of the file:
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@@
 <parts>
 <part name="U$6" library="SparkFun-Boards" deviceset="BEAGLE_BONE_BLACK_CAPE" device=""/>
-<part name="R1" library="rcl" deviceset="R-US_" device="0207/15" value="5K"/>
-<part name="R2" library="rcl" deviceset="R-US_" device="0207/15" value="5K"/>
-<part name="R3" library="rcl" deviceset="R-US_" device="0207/15" value="5K"/>
-<part name="R4" library="rcl" deviceset="R-US_" device="0207/15" value="5K"/>
+<part name="R1" library="rcl" deviceset="R-US_" device="0207/15" value="4.7K"/>
+<part name="R2" library="rcl" deviceset="R-US_" device="0207/15" value="4.7K"/>
+<part name="R3" library="rcl" deviceset="R-US_" device="0207/15" value="4.7K"/>
+<part name="R4" library="rcl" deviceset="R-US_" device="0207/15" value="4.7K"/>
 <part name="B1" library="con-molex" deviceset="87758-1016" device="" value="BUS1-HDR">
 <attribute name="MPN" value="BUS1-HDR"/>
@@
 <text x="149.352" y="87.63" size="1.778" layer="97">Cape GND Rail</text>
 <text x="149.606" y="80.772" size="1.778" layer="97">Cape 3.3V Rail</text>
+<wire x1="76.2" y1="78.74" x2="96.52" y2="78.74" width="0.1524" layer="97"/>
+<wire x1="96.52" y1="78.74" x2="96.52" y2="68.58" width="0.1524" layer="97"/>
+<wire x1="96.52" y1="68.58" x2="76.2" y2="68.58" width="0.1524" layer="97"/>
+<wire x1="76.2" y1="68.58" x2="76.2" y2="78.74" width="0.1524" layer="97"/>
+<text x="83.82" y="66.04" size="1.27" layer="97">Provided on Cape</text>
 </plain>
 <instances>

Commit message: [BB] Updated cape schematic
- All unused wires are now grounded
- I2C pull-up resistor values decreased
- Used another pair of 4.7KΩ resistors in parallel with the built-in
I2C2 pull-ups, making the total pull-up resistance 2.35KΩ
- Reduced I2C1 pull-ups to the closest available value to 2.35KΩ which
is, 2.2KΩ

These changes help with system performance over long bus lengths.
Parts:
- added R5, R6: 4.7K, rcl:R-US_0207/15
- R1, R2: value 4.7K -> 2.2K
Connections:
- net GND: now also B1-2.S, B1-3.S, B1-6.S, B1-7.S, B1-8.S, B1-9.S, B2-2.S, B2-3.S, B2-6.S, B2-7.S, B2-8.S, B2-9.S
- net I2C1_SCL: now also R2.1; no longer R4.1
- net I2C2_SCL: now also R4.1; no longer R3.1
- net I2C2_SDA: now also R3.1; no longer R2.1
Other:
- moved on the sheet: B1-1, B1-10, B1-2, B1-3, B1-4, B1-5, B1-6, B1-7, B1-8, B1-9, B2-1, B2-10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
